Commit message: simple nav implemented

File: src/swarm_prod_sim/resource/bobat.urdf.xacro (robot description, xacro)
@@ -1,6 +1,6 @@
 <?xml version="1.0"?>
-<robot name="/home/kingapiper/Desktop/bobat.urdf" xmlns:xacro="http://ros.org/wiki/xacro">
-  <link name="base_link">
-<!--  <link name="bobat_1_base_link">-->
+<robot name="bobat" xmlns:xacro="http://ros.org/wiki/xacro">
+  <xacro:arg name="robot_id" default="/"/>
+  <link name="$(arg robot_id)base_link">
     <visual>
       <origin xyz="0 0 0.0415" rpy="0 0 0"/>
@@ -17,13 +17,13 @@
   </link>
   <joint name="right wheel motor" type="continuous">
-    <parent link="base_link"/>
-    <child link="right_wheel"/>
+    <parent link="$(arg robot_id)base_link"/>
+    <child link="$(arg robot_id)right_wheel"/>
     <axis xyz="0 1 0"/>
     <limit effort="10" velocity="10"/>
     <origin xyz="0 0 0.025" rpy="-3.141593 0.645101 -3.141593"/>
   </joint>
-  <link name="right_wheel">
+  <link name="$(arg robot_id)right_wheel">
     <visual>
-      <origin xyz="0 -0.045 0" rpy="1.5708 0 0"/>
+      <origin xyz="0 -0.0 0" rpy="1.5708 0 0"/>
       <geometry>
         <cylinder radius="0.025" length="0.01"/>
@@ -31,5 +31,5 @@
     </visual>
     <collision>
-      <origin xyz="0 -0.045 0" rpy="1.5708 0 0"/>
+      <origin xyz="0 -0.0 0" rpy="1.5708 0 0"/>
       <geometry>
         <cylinder radius="0.025" length="0.01"/>
@@ -38,13 +38,13 @@
   </link>
   <joint name="left wheel motor" type="continuous">
-    <parent link="base_link"/>
-    <child link="left_wheel"/>
+    <parent link="$(arg robot_id)base_link"/>
+    <child link="$(arg robot_id)left_wheel"/>
     <axis xyz="0 1 0"/>
     <limit effort="10" velocity="10"/>
     <origin xyz="0 -0.045 0.025" rpy="0 -0.809141 0"/>
   </joint>
-  <link name="left_wheel">
+  <link name="$(arg robot_id)left_wheel">
     <visual>
-      <origin xyz="0 0.045 0" rpy="1.5708 0 0"/>
+      <origin xyz="0 0.0 0" rpy="1.5708 0 0"/>
       <geometry>
         <cylinder radius="0.025" length="0.01"/>
@@ -52,5 +52,5 @@
     </visual>
     <collision>
-      <origin xyz="0 0.045 0" rpy="1.5708 0 0"/>
+      <origin xyz="0 0.0 0" rpy="1.5708 0 0"/>
       <geometry>
         <cylinder radius="0.025" length="0.01"/>
